Commit message: now the urdf has the right joint peoperties. I do need to work on a more realistic mass

File: dexenv/assets/leapXELA_model/robot.urdf (robot description, URDF)
Before this commit: robot leapXELA_model, 21 links, 20 joints
Joints:
- joint if_dip: limit lower=-0.366 upper=2.042 effort=0.95 velocity=8.48 -> lower=-0.366519 upper=2.04204 effort=0.95 velocity=8.48
- joint if_mcp: limit lower=-0.314 upper=2.23 effort=0.95 velocity=8.48 -> lower=-0.314159 upper=2.23402 effort=0.95 velocity=8.48
- joint if_pip: limit lower=-0.506 upper=1.885 effort=0.95 velocity=8.48 -> lower=-0.506145 upper=1.88496 effort=0.95 velocity=8.48
- joint if_rot: limit lower=-1.047 upper=1.047 effort=0.95 velocity=8.48 -> lower=-1.0472 upper=1.0472 effort=0.95 velocity=8.48
- joint mf_dip: limit lower=-0.366 upper=2.042 effort=0.95 velocity=8.48 -> lower=-0.366519 upper=2.04204 effort=0.95 velocity=8.48
- joint mf_mcp: limit lower=-0.314 upper=2.23 effort=0.95 velocity=8.48 -> lower=-0.314159 upper=2.23402 effort=0.95 velocity=8.48
- joint mf_pip: limit lower=-0.506 upper=1.885 effort=0.95 velocity=8.48 -> lower=-0.506145 upper=1.88496 effort=0.95 velocity=8.48
- joint mf_rot: limit lower=-1.047 upper=1.047 effort=0.95 velocity=8.48 -> lower=-1.0472 upper=1.0472 effort=0.95 velocity=8.48
- joint rf_dip: limit lower=-0.366 upper=2.042 effort=0.95 velocity=8.48 -> lower=-0.366519 upper=2.04204 effort=0.95 velocity=8.48
- joint rf_mcp: limit lower=-0.314 upper=2.23 effort=0.95 velocity=8.48 -> lower=-0.314159 upper=2.23402 effort=0.95 velocity=8.48
- joint rf_pip: limit lower=-0.506 upper=1.885 effort=0.95 velocity=8.48 -> lower=-0.506145 upper=1.88496 effort=0.95 velocity=8.48
- joint rf_rot: limit lower=-1.047 upper=1.047 effort=0.95 velocity=8.48 -> lower=-1.0472 upper=1.0472 effort=0.95 velocity=8.48
- joint th_axl: limit lower=-0.47 upper=2.443 effort=0.95 velocity=8.48 -> lower=-0.349066 upper=2.0944 effort=0.95 velocity=8.48
- joint th_cmc: limit lower=-0.349 upper=2.094 effort=0.95 velocity=8.48 -> lower=-0.349066 upper=2.0944 effort=0.95 velocity=8.48
- joint th_ipl: limit lower=-1.34 upper=1.88 effort=0.95 velocity=8.48 -> lower=-1.3439 upper=1.88496 effort=0.95 velocity=8.48
- joint th_mcp: limit lower=-1.20 upper=1.90 effort=0.95 velocity=8.48 -> lower=-0.471239 upper=2.44346 effort=0.95 velocity=8.48
